File: hardware/new_board2/new_board2.kicad_pcb (KiCad board)
At the start: 2 copper layers, 80 x 110 mm, 55 parts, among them CON1 BARREL_JACK, J1 Conn_01x02, J10 Conn_01x02, J11 Conn_01x02, J12 Conn_01x02, J13 Conn_01x02, J14 Conn_01x02, J2 Conn_01x02, J3 Conn_01x02, J4 Conn_01x02, J5 Conn_01x02, J6 Conn_01x02, J7 Conn_01x02, J8 Conn_01x02, J9 Conn_01x02, P1 Conn_01x02, P10 D4, P11 D6, P12 D8, P13 A2, P14 A3, P15 I2C 1, P16 I2C 2, P17 Conn_01x02, P18 Conn_01x02, P2 Conn_01x02, P3 Conn_01x02, P5 Conn_01x02, P6 D7, P7 A1, P8 UART, U1 LM2596T-5, U2 ESP32-DEVKITC-32D

Commit message: pcb version 0.1
Parts:
- removed J10, J11, J12, J13, J14, J2, J3, J4, J5, J6, J8, J9: Conn_01x02, Connector_JST:JST_XH_B2B-XH-A_1x02_P2.50mm_Vertical
- added H1: MountingHole, MountingHole:MountingHole_3.2mm_M3, F.Cu at (139.7, 45.0)
- added H2: MountingHole, MountingHole:MountingHole_3.2mm_M3, F.Cu at (212.3, 45.0)
- added H3: MountingHole, MountingHole:MountingHole_3.2mm_M3, F.Cu at (139.7, 160.0)
- added H4: MountingHole, MountingHole:MountingHole_3.2mm_M3, F.Cu at (212.1, 160.0)
- added P19: Conn_01x02, Connector_PinSocket_2.54mm:PinSocket_1x02_P2.54mm_Vertical, F.Cu at (186.5, 148.0)
- added P20: Conn_01x02, Connector_PinSocket_2.54mm:PinSocket_1x02_P2.54mm_Vertical, F.Cu at (203.5, 117.0)
- added P21: Conn_01x02, Connector_PinSocket_2.54mm:PinSocket_1x02_P2.54mm_Vertical, F.Cu at (203.5, 142.2)
- added P22: Conn_01x02, Connector_PinSocket_2.54mm:PinSocket_1x02_P2.54mm_Vertical, F.Cu at (203.5, 131.8)
- added P4: Conn_01x02, Connector_PinSocket_2.54mm:PinSocket_1x02_P2.54mm_Vertical, F.Cu at (204.0, 58.0)
- added P9: Conn_01x02, Connector_PinSocket_2.54mm:PinSocket_1x02_P2.54mm_Vertical, F.Cu at (204.0, 73.0)
- J1, J7: value Conn_01x02 -> Conn_01x14_Socket; footprint Connector_JST:JST_XH_B2B-XH-A_1x02_P2.50mm_Vertical -> Connector_JST:JST_XH_B14B-XH-A_1x14_P2.50mm_Vertical
- P17, P18, P3, P5: footprint Connector_JST:JST_XH_B2B-XH-A_1x02_P2.50mm_Vertical -> Connector_PinSocket_2.54mm:PinSocket_1x02_P2.54mm_Vertical
- moved J1 91.8 mm to (141.0, 52.5)
- moved P2 50.0 mm to (147.4, 154.9), turned to 0 degrees
- moved J7 43.5 mm to (141.0, 114.5), turned to -90 degrees
- moved P1 37.8 mm to (156.7, 154.8), turned to 0 degrees
- moved R6 18.9 mm to (156.7, 121.7)
- moved R2 14.3 mm to (156.8, 131.1)
- moved R7 4.83 mm to (156.8, 140.6)
- moved R5 4.75 mm to (156.9, 135.8)
- moved R3 4.66 mm to (156.8, 116.8)
- moved P3 2.89 mm to (204.0, 86.5), turned to 180 degrees
- moved P18 2.30 mm to (204.0, 102.2), turned to 180 degrees
- moved P5 0.33 mm to (203.0, 148.0), turned to -90 degrees
- moved R4 0.24 mm to (156.8, 126.5)
Connections:
- net Net-(P1-Pin_1) renamed +12V
- J1 pad 1: Net-(J1-Pin_1) -> +3V3
- J1 pad 2: GND -> +3V3
- J7 pad 1: Net-(J7-Pin_1) -> GND
- P13 pad 3: +5V -> Net-(P13-Pin_3)
- P14 pad 3: +5V -> Net-(P14-Pin_3)
- P15 pad 3: +5V -> Net-(P15-Pin_3)
- P16 pad 3: +5V -> Net-(P16-Pin_3)
- P7 pad 3: +5V -> Net-(P22-Pin_1)
- P8 pad 3: +5V -> Net-(P19-Pin_1)
- R17 pad 2: Net-(J14-Pin_1) -> Net-(J7-Pin_8)
- R2 pad 2: Net-(J4-Pin_1) -> Net-(J7-Pin_12)
- R3 pad 2: Net-(J5-Pin_1) -> Net-(J7-Pin_9)
- R4 pad 2: Net-(J1-Pin_1) -> Net-(J7-Pin_11)
- R5 pad 2: Net-(J6-Pin_1) -> Net-(J7-Pin_13)
- R6 pad 2: Net-(J7-Pin_1) -> Net-(J7-Pin_10)
- R7 pad 2: Net-(J8-Pin_1) -> Net-(J7-Pin_14)
Routing:
- net +5V: track 401.4 -> 462.5 mm
- net +3V3: track 87.1 -> 57.2 mm
- net Net-(J6-Pin_1): track 25.0 -> 0.00 mm
- net Net-(J7-Pin_8): track 0.00 -> 23.8 mm
- net +12V: track 193.5 -> 216.6 mm
- net Net-(J1-Pin_1): track 20.9 -> 0.00 mm
- net Net-(J8-Pin_1): track 20.9 -> 0.00 mm
- net Net-(J7-Pin_9): track 0.00 -> 20.5 mm
- net Net-(J7-Pin_1): track 18.1 -> 0.00 mm
- net Net-(J7-Pin_10): track 0.00 -> 18.1 mm
- net D6-3: track 39.6 -> 22.2 mm
- net D4-3: track 121.6 -> 104.6 mm
- net Net-(J5-Pin_1): track 16.6 -> 0.00 mm
- net Net-(J7-Pin_11): track 0.00 -> 15.8 mm
- net Net-(J7-Pin_12): track 0.00 -> 13.8 mm
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Other:
- board size 80 x 110 mm -> 80.7 x 123.4 mm
- board text added: "5-choice-serial-test v0.1"
