File: hardware/new_board2/new_board2.kicad_sch (KiCad schematic)
At the start: 60 parts, among them CON1 BARREL_JACK, J1 Conn_01x06_Socket, J10 Conn_01x02, J11 Conn_01x02, J12 Conn_01x02, J13 Conn_01x02, J14 Conn_01x02, J2 Conn_01x02, J3 Conn_01x02, J4 Conn_01x06_Socket, J5 Conn_01x06_Socket, J6 Conn_01x06_Socket, J7 Conn_01x14_Socket, J9 Conn_01x02, P10 A2, P11 A3, P12 UART, P13 I2C 1, P14 I2C 2, P15 Conn_01x02, P16 Conn_01x02, P17 Conn_01x02, P18 Conn_01x02, P19 Conn_01x02, P20 Conn_01x02, P21 Conn_01x02, P22 Conn_01x02, P3 Conn_01x02, P4 Conn_01x02, P4 D4, P5 Conn_01x02, P6 D6, P7 D7, P8 D8, P9 A1, P9 Conn_01x02, U1 LM2596T-5, U3 ESP32-DEVKITC-32D

Commit message: update new board
Parts:
- removed J1, J4, J5, J6: Conn_01x06_Socket, symbol Connector:Conn_01x06_Socket
- removed J10, J11, J12, J13, J14, J2, J3, J9: Conn_01x02, Connector_JST:JST_XH_B2B-XH-A_1x02_P2.50mm_Vertical, symbol Connector_Generic:Conn_01x02
- added J1: Conn_01x14_Socket, Connector_JST:JST_XH_B14B-XH-A_1x14_P2.50mm_Vertical, symbol Connector:Conn_01x14_Socket
- J7: footprint (none) -> Connector_JST:JST_XH_B14B-XH-A_1x14_P2.50mm_Vertical
- P10, P11, P12, P13, P14, P4, P6, P7, P8, P9: footprint Connector_JST:JST_XH_B4B-XH-A_1x04_P2.50mm_Vertical -> Connector_PinSocket_2.54mm:PinSocket_1x02_P2.54mm_Vertical
- P17, P18, P19, P20, P21, P22, P3, P4, P5, P9: footprint Connector_JST:JST_XH_B2B-XH-A_1x02_P2.50mm_Vertical -> Connector_PinSocket_2.54mm:PinSocket_1x02_P2.54mm_Vertical
Connections:
- net +3V3: now also J1.1 (Pin_1), J1.2 (Pin_2), J1.3 (Pin_3), J1.4 (Pin_4), J1.5 (Pin_5), J1.6 (Pin_6), J1.7 (Pin_7)
- net D1-3: now also J1.8 (Pin_8)
- net D1-4: now also J1.9 (Pin_9)
- net D3-3: now also J1.10 (Pin_10)
- net D3-4: now also J1.11 (Pin_11)
- net D5-3: now also J1.12 (Pin_12)
- net D5-4: now also J1.13 (Pin_13)
- net D6-3: now also J1.14 (Pin_14)
- net GND: now also J7.1 (Pin_1), J7.2 (Pin_2), J7.3 (Pin_3), J7.4 (Pin_4), J7.5 (Pin_5), J7.6 (Pin_6), J7.7 (Pin_7)
- net at R6.2: now also J7.10 (Pin_10)
- net +12V: now reaches C1.1, CON1.1, P15.1 (Pin_1), P16.1 (Pin_1), R1.2, U1.1 (VIN)
- net at R17.2: now also J7.8 (Pin_8)
- net at J7.11 (Pin_11): now also R4.2
- net at J7.12 (Pin_12): now also R2.2
- net at J7.13 (Pin_13): now also R5.2
- net at J7.14 (Pin_14): now also R7.2
- net at J7.9 (Pin_9): now also R3.2
Other:
- moved on the sheet: J7, R17, R2, R3, R4, R5, R6, R7

Commit message: add first version of new board
Parts:
- renumbered J7 to J1, J1 to J2, P21 to P13, P5 to P14, P17 to P15, P18 to P16, P20 to P18, P9 to P21, P4 to P22, P3 to P6, P22 to P7, P19 to P8, R5 to R10, R10 to R11, R11 to R12, R12 to R13, R13 to R14, R14 to R16, R16 to R17, R8 to R2, R9 to R3, R3 to R5, R17 to R7, R2 to R8, R7 to R9
