File: hardware/Schematics/new_board2/new_board2.kicad_pcb (KiCad board)
At the start: 2 copper layers, 80.7 x 123.4 mm, 53 parts, among them CON1 BARREL_JACK, J1 Conn_01x14_Socket, J7 Conn_01x14_Socket, P1 Conn_01x02, P10 D4, P11 D6, P12 D8, P13 A2, P14 A3, P15 I2C 1, P16 I2C 2, P17 Conn_01x02, P18 Conn_01x02, P19 Conn_01x02, P2 Conn_01x02, P20 Conn_01x02, P21 Conn_01x02, P22 Conn_01x02, P3 Conn_01x02, P4 Conn_01x02, P5 Conn_01x02, P6 D7, P7 A1, P8 UART, P9 Conn_01x02, U1 LM2596T-5, U2 ESP32-DEVKITC-32D

Commit message: Documentation update
Parts:
- renumbered J7 to J1, J1 to J2, P11 to P10, P12 to P11, P13 to P12, P21 to P13, P5 to P14, P17 to P15, P18 to P16, P14 to P17, P20 to P18, P15 to P19, P16 to P20, P9 to P21, P4 to P22, P6 to P3, P7 to P4, P8 to P5, P3 to P6, P22 to P7, P19 to P8, P10 to P9, R5 to R10, R10 to R11, R11 to R12, R12 to R13, R13 to R14, R14 to R16, R16 to R17, R8 to R2, R9 to R3, R3 to R5, R17 to R7, R2 to R8, R7 to R9
Other:
- board text removed: "BeeHive v0.7"
- board text removed: "IO15"
- board text removed: "IO16"
- board text removed: "IO17"
- board text removed: "IO19"
- board text removed: "IO2"
- board text removed: "IO21"
- board text removed: "IO22"
- board text removed: "IO23"
- board text removed: "IO36"
- board text removed: "IO39"
