File: hardware/Schematics/new_board2/new_board2.kicad_sch (KiCad schematic)
At the start: 53 parts, among them CON1 BARREL_JACK, J1 Conn_01x14_Socket, J2 Conn_01x14_Socket, P10 A2, P11 A3, P12 UART, P13 Conn_01x02, P13 I2C 1, P14 Conn_01x02, P14 I2C 2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

Commit message: Documentation update
Changed lines of the file:
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@@
 				)
 				(justify left bottom)
-				(hide yes)
 			)
 		)
