File: hardware/printed_circuit_board/new_board2/new_board2.kicad_sch (KiCad schematic)
At the start: 53 parts, among them CON1 BARREL_JACK, J1 Conn_01x14_Socket, J2 Conn_01x14_Socket, P10 A2, P11 A3, P12 UART, P13 Conn_01x02, P13 I2C 1, P14 Conn_01x02, P14 I2C 2, P15 Conn_01x02, P16 Conn_01x02, P18 Conn_01x02, P21 Conn_01x02, P22 Conn_01x02, P4 D4, P6 Conn_01x02, P6 D6, P7 Conn_01x02, P7 D7, P8 Conn_01x02, P8 D8, P9 A1, U1 LM2596T-5, U3 ESP32-DEVKITC-32D

Commit message: simplify PCB, making stable connections for LEDs using a ULN2003, remove jumpers, THIS IS STILL UNTESTED!
Parts:
- removed P11: A3, Connector_JST:JST_XH_B4B-XH-A_1x04_P2.50mm_Vertical, symbol Connector_Generic:Conn_01x04
- removed P13, P14, P15, P16, P18, P21, P22, P6, P7, P8: Conn_01x02, Connector_PinSocket_2.54mm:PinSocket_1x02_P2.54mm_Vertical, symbol Connector_Generic:Conn_01x02
- removed P7: D7, Connector_JST:JST_XH_B4B-XH-A_1x04_P2.50mm_Vertical, symbol Connector_Generic:Conn_01x04
- removed P8: D8, Connector_JST:JST_XH_B4B-XH-A_1x04_P2.50mm_Vertical, symbol Connector_Generic:Conn_01x04
- removed P9: A1, Connector_JST:JST_XH_B4B-XH-A_1x04_P2.50mm_Vertical, symbol Connector_Generic:Conn_01x04
- added J3: Conn_01x14_Socket, Connector_JST:JST_XH_B14B-XH-A_1x14_P2.50mm_Vertical, symbol Connector:Conn_01x14_Socket
- added R18, R20, R21, R22, R23, R24, R25: 560, Resistor_THT:R_Box_L13.0mm_W4.0mm_P9.00mm, symbol Device:R
- added U3: ULN2003, Package_DIP:DIP-16_W7.62mm_Socket_LongPads, symbol Transistor_Array:ULN2003
Connections:
- net +5V: now also P10.3 (Pin_3), P12.3 (Pin_3), P13.3 (Pin_3), P14.3 (Pin_3), P4.3 (Pin_3), P6.3 (Pin_3), J3.1 (Pin_1), J3.2 (Pin_2), J3.3 (Pin_3), J3.4 (Pin_4), J3.5 (Pin_5), J3.6 (Pin_6), J3.7 (Pin_7)
- net GND: now also U3.8 (GND)
- net A1-3: no longer names the net of U3.6 (IO35)
- net A1-3: now also U3.7 (I7)
- net A1-4: no longer names the net of U3.5 (IO34)
- net A3-3: no longer names the net of U3.7 (IO32)
- net A3-3: now also U3.6 (I6)
- net A3-4: no longer names the net of U3.8 (IO33)
- net A3-4: now also U3.5 (I5)
- net D7-3: no longer names the net of U3.12 (IO14)
- net D7-3: now also U3.1 (I1)
- net D7-4: no longer names the net of U3.11 (IO27)
- net D7-4: now also U3.2 (I2)
- net D8-3: no longer names the net of U3.10 (IO26)
- net D8-3: now also U3.3 (I3)
- net D8-4: no longer names the net of U3.9 (IO25)
- net D8-4: now also U3.4 (I4)
- new net: J3.13 (Pin_13), R25.1
- new net: R25.2, U3.11 (O6)
- new net: J3.12 (Pin_12), R24.1
- new net: R24.2, U3.12 (O5)
- new net: J3.14 (Pin_14), R18.1
- new net: R18.2, U3.10 (O7)
- new net: J3.9 (Pin_9), R21.1
- new net: R21.2, U3.15 (O2)
- new net: J3.11 (Pin_11), R23.1
- new net: R23.2, U3.13 (O4)
- new net: J3.10 (Pin_10), R22.1
- new net: R22.2, U3.14 (O3)
- new net: R20.2, U3.16 (O1)
- new net: J3.8 (Pin_8), R20.1
- no-connect marks 10 -> 11
Other:
- moved on the sheet: J1, J2, P10, P12, P13, P14, R10, R11, R12, R13, R14, R15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
